Commit message: changed torque

File: Project2/my_robot/urdf/my_robot.xacro (robot description, xacro)
@@ -31,28 +31,4 @@
       </geometry>
     </visual>
-    <collision name='back_caster_collision'>
-      <origin xyz="-0.3 0 -0.05" rpy=" 0 0 0"/>
-      <geometry>
-        <sphere radius="0.1"/>
-      </geometry>
-    </collision>
-    <visual name='back_caster_visual'>
-      <origin xyz="-0.3 0 -0.05" rpy=" 0 0 0"/>
-      <geometry>
-        <sphere radius="0.1"/>
-      </geometry>
-    </visual>
-    <collision name='front_caster_collision'>
-      <origin xyz="0.3 0 -0.05" rpy=" 0 0 0"/>
-      <geometry>
-        <sphere radius="0.1"/>
-      </geometry>
-    </collision>
-    <visual name='front_caster_visual'>
-      <origin xyz="0.3 0 -0.05" rpy=" 0 0 0"/>
-      <geometry>
-        <sphere radius="0.1"/>
-      </geometry>
-    </visual>
   </link>
   <link name="front_left_wheel">
